Commit message: updates

File: gimbal_urdf/urdf/gimbal.urdf.xacro (robot description, xacro)
@@ -35,5 +35,5 @@
         </material>
       </visual>
-      <collision>
+      <!-- <collision>
         <origin
           xyz="0 0 0"
@@ -43,5 +43,5 @@
             filename="package://gimbal_urdf/meshes/base_link.STL" />
         </geometry>
-      </collision>
+      </collision> -->
     </link>
     <link
@@ -75,5 +75,5 @@
         </material>
       </visual>
-      <collision>
+      <!-- <collision>
         <origin
           xyz="0 0 0"
@@ -83,5 +83,5 @@
             filename="package://gimbal_urdf/meshes/mid_link.STL" />
         </geometry>
-      </collision>
+      </collision> -->
     </link>
     <joint
@@ -133,5 +133,5 @@
         </material>
       </visual>
-      <collision>
+      <!-- <collision>
         <origin
           xyz="0 0 0"
@@ -141,5 +141,5 @@
             filename="package://gimbal_urdf/meshes/dist_link.STL" />
         </geometry>
-      </collision>
+      </collision> -->
     </link>
     <joint
@@ -154,5 +154,5 @@
         link="dist_link" />
       <axis
-        xyz="0 0 1" />
+        xyz="0 0 -1" />
       <limit
         lower="0"
@@ -161,4 +161,17 @@
         velocity="0" />
     </joint>
+     <ros2_control name="gimbal_ros2_control" type="system">
+      <hardware>
+      <plugin>mock_components/GenericSystem</plugin>
+      </hardware>
+      <joint name="mid_joint">
+      <state_interface name="position">
+      </state_interface>
+      </joint>
+      <joint name="dist_joint">
+      <state_interface name="position">
+      </state_interface>
+      </joint>
+     </ros2_control>
   </xacro:macro>
 </robot>

File: gimbal_urdf/urdf/gimbal_urdf.urdf (robot description, URDF)
Before this commit: robot gimbal_urdf, 3 links, 2 joints
Joints:
- joint mid_joint: limit lower=0 upper=0 effort=0 velocity=0 -> lower=0 upper=0 effort=2 velocity=2

File: gimbal_urdf/urdf/ur_gimbal.urdf.xacro (robot description, xacro)
@@ -7,5 +7,5 @@
    <!-- possible 'ur_type' values: ur3, ur3e, ur5, ur5e, ur10, ur10e, ur16e, ur20, ur30 -->
    <!-- the default value should raise an error in case this was called without defining the type -->
-   <xacro:arg name="ur_type" default="ur5e"/>
+   <xacro:arg name="ur_type" default="ur5x"/>
    <!-- parameters -->
    <xacro:arg name="tf_prefix" default="" />
@@ -18,9 +18,37 @@
    <xacro:arg name="safety_pos_margin" default="0.15"/>
    <xacro:arg name="safety_k_position" default="20"/>
-   <!--When using gazebo simulations absolute paths are necessary.-->
-   <xacro:arg name="force_abs_paths" default="false" />
+   <!-- ros2_control related parameters -->
+   <xacro:arg name="headless_mode" default="false" />
+   <xacro:arg name="robot_ip" default="0.0.0.0" />
+   <xacro:arg name="script_filename" default=""/>
+   <xacro:arg name="output_recipe_filename" default=""/>
+   <xacro:arg name="input_recipe_filename" default=""/>
+   <xacro:arg name="reverse_ip" default="0.0.0.0"/>
+   <xacro:arg name="script_command_port" default="50004"/>
+   <xacro:arg name="reverse_port" default="50001"/>
+   <xacro:arg name="script_sender_port" default="50002"/>
+   <xacro:arg name="trajectory_port" default="50003"/>
+   <!--   tool communication related parameters-->
+   <xacro:arg name="use_tool_communication" default="false" />
+   <xacro:arg name="tool_voltage" default="0" />
+   <xacro:arg name="tool_parity" default="0" />
+   <xacro:arg name="tool_baud_rate" default="115200" />
+   <xacro:arg name="tool_stop_bits" default="1" />
+   <xacro:arg name="tool_rx_idle_chars" default="1.5" />
+   <xacro:arg name="tool_tx_idle_chars" default="3.5" />
+   <xacro:arg name="tool_device_name" default="/tmp/ttyUR" />
+   <xacro:arg name="tool_tcp_port" default="54321" />
+     <!-- Simulation parameters -->
+   <xacro:arg name="use_fake_hardware" default="false" />
+   <xacro:arg name="fake_sensor_commands" default="false" />
+   <xacro:arg name="sim_gazebo" default="false" />
+   <xacro:arg name="sim_ignition" default="false" />
+   <xacro:arg name="simulation_controllers" default="" />
+   <!-- initial position for simulations (Fake Hardware, Gazebo, Ignition) -->
+   <xacro:arg name="initial_positions_file" default="$(find ur_description)/config/initial_positions.yaml"/>
+   <!-- convert to property to use substitution in function -->
+   <xacro:property name="initial_positions_file" default="$(arg initial_positions_file)"/>
    <!-- create link fixed to the "world" -->
    <link name="world" />
-   <xacro:include filename="$(find gimbal_urdf)/urdf/gimbal.urdf.xacro" />
    <!-- arm -->
    <xacro:ur_robot
@@ -32,17 +60,64 @@
      physical_parameters_file="$(arg physical_params)"
      visual_parameters_file="$(arg visual_params)"
+     transmission_hw_interface="$(arg transmission_hw_interface)"
      safety_limits="$(arg safety_limits)"
      safety_pos_margin="$(arg safety_pos_margin)"
      safety_k_position="$(arg safety_k_position)"
+     use_fake_hardware="$(arg use_fake_hardware)"
+     fake_sensor_commands="$(arg fake_sensor_commands)"
+     sim_gazebo="$(arg sim_gazebo)"
+     sim_ignition="$(arg sim_ignition)"
+     headless_mode="$(arg headless_mode)"
+     initial_positions="${xacro.load_yaml(initial_positions_file)}"
+     use_tool_communication="$(arg use_tool_communication)"
+     tool_voltage="$(arg tool_voltage)"
+     tool_parity="$(arg tool_parity)"
+     tool_baud_rate="$(arg tool_baud_rate)"
+     tool_stop_bits="$(arg tool_stop_bits)"
+     tool_rx_idle_chars="$(arg tool_rx_idle_chars)"
+     tool_tx_idle_chars="$(arg tool_tx_idle_chars)"
+     tool_device_name="$(arg tool_device_name)"
+     tool_tcp_port="$(arg tool_tcp_port)"
+     robot_ip="$(arg robot_ip)"
+     script_filename="$(arg script_filename)"
+     output_recipe_filename="$(arg output_recipe_filename)"
+     input_recipe_filename="$(arg input_recipe_filename)"
+     reverse_ip="$(arg reverse_ip)"
+     script_command_port="$(arg script_command_port)"
+     reverse_port="$(arg reverse_port)"
+     script_sender_port="$(arg script_sender_port)"
+     trajectory_port="$(arg trajectory_port)"
      >
      <origin xyz="0 0 0" rpy="0 0 0" />          <!-- position robot in the world -->
    </xacro:ur_robot>
+   <xacro:if value="$(arg sim_gazebo)">
+    <!-- Gazebo plugins -->
+    <gazebo reference="world">
+    </gazebo>
+    <gazebo>
+      <plugin filename="libgazebo_ros2_control.so" name="gazebo_ros2_control">
+        <parameters>$(arg simulation_controllers)</parameters>
+      </plugin>
+    </gazebo>
+  </xacro:if>
+  <xacro:if value="$(arg sim_ignition)">
+    <!-- Gazebo plugins -->
+    <gazebo reference="world">
+    </gazebo>
+    <gazebo>
+      <plugin filename="libign_ros2_control-system.so" name="ign_ros2_control::IgnitionROS2ControlPlugin">
+        <parameters>$(arg simulation_controllers)</parameters>
+        <controller_manager_node_name>$(arg tf_prefix)controller_manager</controller_manager_node_name>
+      </plugin>
+    </gazebo>
+  </xacro:if>
+  <xacro:include filename="$(find gimbal_urdf)/urdf/gimbal.urdf.xacro" />
+  <joint name="gimbal_mount" type="fixed">
+    <origin xyz="0 0 0" rpy="0 -1.57 0" />
+    <parent link="$(arg tf_prefix)tool0" />
+    <child link="gimbal_base_link" />
+  </joint>
   <xacro:gimbal_macro />
     <!-- <origin xyz="0 0 0" rpy="0 0 0" /> -->
   <!-- </xacro:gimble_macro> -->
-  <joint name="gimbal_mount" type="fixed">
-    <origin xyz="0 0 0" rpy="0 0 0" />
-    <parent link="$(arg tf_prefix)tool0" />
-    <child link="gimbal_base_link" />
-  </joint>
 </robot>
